File: LEDPoet.brd (EAGLE design)
At the start: 50 x 25 mm, 27 parts, among them IC1 PIC12F1822, U1 FAN5333

Commit message: gerber done
Parts:
- moved JP4 39.3 mm to (46.4, 11.2)
- moved C6 32.1 mm to (27.9, 7.62)
- moved C5 31.4 mm to (21.6, 7.62)
- moved D3 31.4 mm to (21.6, 5.08)
- moved L1 31.4 mm to (21.6, 11.4)
- moved R6 31.4 mm to (26.7, 16.5)
- moved U1 31.4 mm to (21.6, 16.5)
- moved D1 30.3 mm to (26.7, 11.4)
- moved C1 18.4 mm to (36.2, 2.54), turned to 90 degrees
- moved S1 14.0 mm to (36.8, 12.5), turned to 90 degrees
- moved R10 13.3 mm to (34.3, 2.54), turned to 270 degrees
- moved R9 8.25 mm to (32.4, 2.54), turned to 270 degrees
- moved R1 6.99 mm to (14.6, 6.35)
- moved C4 6.35 mm to (16.5, 6.35)
- moved R3 6.35 mm to (12.7, 6.35)
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Routing:
- net VCC: track 0.00 -> 55.0 mm, vias 0 -> 2
- net SWITCH: track 0.00 -> 31.2 mm, vias 0 -> 2
- net V+: track 0.00 -> 29.4 mm
- net LED-: track 0.00 -> 25.0 mm
- net /RST: track 0.00 -> 22.8 mm, vias 0 -> 2
- net LED+: track 0.00 -> 20.1 mm
- net N$6: track 0.00 -> 17.4 mm
- net GND: track 0.00 -> 17.0 mm, vias 0 -> 17
- net ICSPCLK: track 0.00 -> 9.19 mm
- net LED: track 0.00 -> 8.49 mm
- net N$7: track 0.00 -> 7.88 mm, vias 0 -> 1
- net ICSPDAT: track 0.00 -> 7.83 mm
- net N$4: track 0.00 -> 7.34 mm
- net N$3: track 0.00 -> 3.42 mm
- net N$2: track 0.00 -> 1.90 mm
- added copper zone on layer 1, net GND
- added copper zone on layer 16, net GND
- added copper zone on layer 1, net LED+
- added copper zone on layer 1, net N$5
- added copper zone on layer 1, net V+
Other:
- outline, holes or cut-outs redrawn
- board text added: "ANTICLIMAX"
- board text added: "LED Poet"
